Commit message: fix diff plugin transformation and dummy link joint

File: src/robot_description/urdf/ajrobot.xacro (robot description, xacro)
@@ -31,6 +31,6 @@
 <!-- Fixed joint connecting base_footprint -> base_link -->
 <joint name="base_footprint_joint" type="fixed">
-  <parent link="base_footprint"/>
-  <child link="base_link"/>
+  <parent link="base_link"/>
+  <child link="base_footprint"/>
   <origin xyz="0 0 0" rpy="0 0 0"/>
 </joint>

Commit message: fixed ajrobot kinematics

File: src/robot_description/urdf/ajrobot.xacro (robot description, xacro)
@@ -11,7 +11,7 @@
 <link name="base_link">
   <inertial>
-    <origin rpy="0 0 0" xyz="-0.00189 0.00078 0.0875"/>
-    <mass value="14.612"/>
-    <inertia ixx="0.0539" ixy="-1e-06" ixz="-0.00045" iyy="0.0564" iyz="-1e-06" izz="0.04208"/>
+    <origin rpy="0 0 0" xyz="-0.0018939651836912175 0.0007828486855805901 0.08750494563386604"/>
+    <mass value="14.612879724425715"/>
+    <inertia ixx="0.053945" ixy="-1e-06" ixz="-0.000455" iyy="0.056464" iyz="-1e-06" izz="0.04208"/>
   </inertial>
   <visual>

Commit message: add imu

File: src/robot_description/urdf/ajrobot.xacro (robot description, xacro)
@@ -6,4 +6,12 @@
 <xacro:include filename="$(find robot_description)/gazebo/ajrobot_detailed_physics.gazebo" />
 <xacro:include filename="$(find robot_description)/gazebo/ajrobot_detailed_plugins.gazebo" />
+<!-- Define inertial property macros  -->
+<xacro:macro name="box_inertia" params="m w h d">
+  <inertial>
+    <origin xyz="0 0 0" rpy="${pi/2} 0 ${pi/2}"/>
+    <mass value="${m}"/>
+    <inertia ixx="${(m/12) * (h*h + d*d)}" ixy="0.0" ixz="0.0" iyy="${(m/12) * (w*w + d*d)}" iyz="0.0" izz="${(m/12) * (w*w + h*h)}"/>
+  </inertial>
+</xacro:macro>
 <!-- Dummy root link (base_footprint) -->
 <link name="base_footprint" />
@@ -35,4 +43,21 @@
   <origin xyz="0 0 0" rpy="0 0 0"/>
 </joint>
+<link name="imu_link">
+  <visual>
+    <geometry>
+      <!-- Keep small size but move position -->
+      <box size="0.02 0.02 0.02"/>
+    </geometry>
+    <material name="red">
+      <color rgba="1 0 0 1"/>
+    </material>
+  </visual>
+  <collision>
+    <geometry>
+      <box size="0.02 0.02 0.02"/>
+    </geometry>
+  </collision>
+  <xacro:box_inertia m="0.01" w="0.02" d="0.02" h="0.02"/>
+</link>
 <link name="rwheel_1">
   <inertial>
@@ -255,4 +280,10 @@
   </collision>
 </link>
+<link name="camera_depth_frame"/>
+<joint name="camera_depth_joint" type="fixed">
+  <origin xyz="-0.052209 -0.000782 -0.071425" rpy="${-pi/2} 0 ${-pi/2}"/>
+  <parent link="camera_1"/>
+  <child link="camera_depth_frame"/>
+</joint>
 <link name="pir_1">
   <inertial>
@@ -275,4 +306,9 @@
   </collision>
 </link>
+<joint name="imu_joint" type="fixed">
+  <parent link="base_link"/>
+  <child link="imu_link"/>
+  <origin xyz="0 0 0.05"/>
+</joint>
 <joint name="rwheel_joint" type="continuous">
   <origin rpy="0 0 0" xyz="0.000209 -0.068118 0.027225"/>
